Commit message: change the simulation env

File: lbr_description/urdf/iiwa14/iiwa14_description.xacro (robot description, xacro)
@@ -400,4 +400,5 @@
         <parent link="base"/>
         <child link="mount"/>
+        <origin xyz="0 0 0" rpy="0 0 -1.57"/>
     </joint>
     <link name="mount">
@@ -405,5 +406,5 @@
             <origin xyz="0 0 0.145" rpy="0 0 0"/>
             <geometry>
-                <mesh filename="package://lbr_description/meshes/envs/visual/mount.dae"/>
+                <mesh filename="package://lbr_description/meshes/envs/visual/mount.stl"/>
             </geometry>
             <material name="gray">
@@ -519,5 +520,5 @@
         <parent link="$(arg robot_name)_floating_link"/>
         <child link = "iiwa2"/>
-        <origin xyz="0 0 0.94" rpy="1.57 0 0"/>
+        <origin xyz="-0.005 -0.0045 0.94" rpy="1.57 0 0"/>
     </joint>
     <link name="iiwa2">
