Commit message: update lbr_description

File: lbr_description/urdf/iiwa14/iiwa14.xacro (robot description, xacro)
@@ -11,5 +11,5 @@
     <!-- KDL requires a link without inertia -->
     <link name="$(arg robot_name)_floating_link" />
-    <link name="workspace_mount">
+    <link name="workspace_mount1">
         <visual>
             <origin xyz="0 0 0" rpy="0 0 0"/>
@@ -28,12 +28,12 @@
         </collision>
     </link>
-    <joint name="workspace_mount_joint" type="fixed">
-        <origin xyz="0.1 1.14 0.85" rpy="0 0 3.14"/>
+    <joint name="workspace_mount1_joint" type="fixed">
+        <origin xyz="0.1 0.5 0.85" rpy="0 0 3.14"/>
         <parent link="$(arg robot_name)_floating_link"/>
-        <child link="workspace_mount"/>
+        <child link="workspace_mount1"/>
     </joint>
     <joint name="$(arg robot_name)_joint" type="fixed">
         <origin xyz="0 0 0.016" rpy="0 0 0.785398"/>
-        <parent link="workspace_mount" />
+        <parent link="workspace_mount1" />
         <child link="$(arg robot_name)_link_0" />
     </joint>

File: lbr_description/urdf/iiwa14/iiwa14_description.xacro (robot description, xacro)
@@ -368,13 +368,14 @@
     <!--  The TCP frame is here defined -->
     <link name="tool_link_ee"/>
-    <joint name="base_joint" type="fixed">
+    <joint name="conveyor_joint" type="fixed">
         <parent link="$(arg robot_name)_floating_link"/>
-        <child link="base"/>
-    </joint>
-    <link name="base">
-        <visual>
-            <origin xyz="0 0 0" rpy="0 0 0"/>
-            <geometry>
-                <mesh filename="package://lbr_description/meshes/envs/visual/base.dae"/>
+        <child link = "conveyor"/>
+        <origin xyz="0.6 1.7 0" rpy="0 0 0"/>
+    </joint>
+    <link name="conveyor">
+        <visual>
+            <origin xyz="0 0 0" rpy="0 0 0"/>
+            <geometry>
+                <mesh filename="package://lbr_description/meshes/envs/visual/conveyor.dae"/>
             </geometry>
             <material name="gray">
@@ -383,7 +384,7 @@
         </visual>
         <collision>
-            <origin xyz="0 0 0.06" rpy="0 0 0"/>
-            <geometry>
-                <box size="0.4 0.4 0.10"/>
+            <origin xyz="0 0 0.455" rpy="0 0 0"/>
+            <geometry>
+                <box size="0.445 3.0 0.91"/>
             </geometry>
         </collision>
@@ -397,14 +398,14 @@
         </inertial>
     </link>
-    <joint name="mount_joint" type="fixed">
-        <parent link="base"/>
-        <child link="mount"/>
-        <origin xyz="0 0 0" rpy="0 0 -1.57"/>
-    </joint>
-    <link name="mount">
-        <visual>
-            <origin xyz="0 0 0.145" rpy="0 0 0"/>
-            <geometry>
-                <mesh filename="package://lbr_description/meshes/envs/visual/mount.stl"/>
+    <joint name="tv_joint" type="fixed">
+        <parent link="$(arg robot_name)_floating_link"/>
+        <child link = "tv"/>
+        <origin xyz="0.6 -0.5 1.9" rpy="-0.1745 0 0.78"/>
+    </joint>
+    <link name="tv">
+        <visual>
+            <origin xyz="0 0 0" rpy="0 0 0"/>
+            <geometry>
+                <box size="1.1 0.1 0.6"/>
             </geometry>
             <material name="gray">
@@ -413,7 +414,7 @@
         </visual>
         <collision>
-            <origin xyz="0 0 0.565" rpy="0 0 0"/>
-            <geometry>
-                <box size="0.25 0.25 0.82"/>
+            <origin xyz="0 0 0" rpy="0 0 0"/>
+            <geometry>
+                <box size="1.1 0.1 0.6"/>
             </geometry>
         </collision>
@@ -427,14 +428,14 @@
         </inertial>
     </link>
-    <joint name="conveyor_joint" type="fixed">
+    <joint name="frame_joint" type="fixed">
         <parent link="$(arg robot_name)_floating_link"/>
-        <child link = "conveyor"/>
-        <origin xyz="0.6 1.7 0" rpy="0 0 0"/>
-    </joint>
-    <link name="conveyor">
-        <visual>
-            <origin xyz="0 0 0" rpy="0 0 0"/>
-            <geometry>
-                <mesh filename="package://lbr_description/meshes/envs/visual/conveyor.dae"/>
+        <child link = "frame"/>
+        <origin xyz="-0.2 0.8 0.84" rpy="0 0 0"/>
+    </joint>
+    <link name="frame">
+        <visual>
+            <origin xyz="0 0 0" rpy="0 0 0"/>
+            <geometry>
+                <mesh filename="package://lbr_description/meshes/envs/visual/workspace.stl"/>
             </geometry>
             <material name="gray">
@@ -443,7 +444,7 @@
         </visual>
         <collision>
-            <origin xyz="0 0 0.455" rpy="0 0 0"/>
-            <geometry>
-                <box size="0.445 3.0 0.91"/>
+            <origin xyz="0 0 -0.4" rpy="0 0 0"/>
+            <geometry>
+                <box size="1.0 1.0 0.7"/>
             </geometry>
         </collision>
@@ -457,14 +458,9 @@
         </inertial>
     </link>
-    <joint name="tv_joint" type="fixed">
-        <parent link="$(arg robot_name)_floating_link"/>
-        <child link = "tv"/>
-        <origin xyz="0.6 -0.9 1.9" rpy="-0.1745 0 0.78"/>
-    </joint>
-    <link name="tv">
-        <visual>
-            <origin xyz="0 0 0" rpy="0 0 0"/>
-            <geometry>
-                <box size="1.1 0.1 0.6"/>
+    <link name="workspace_mount2">
+        <visual>
+            <origin xyz="0 0 0" rpy="0 0 0"/>
+            <geometry>
+                <box size="0.3 0.3 0.03"/>
             </geometry>
             <material name="gray">
@@ -475,5 +471,32 @@
             <origin xyz="0 0 0" rpy="0 0 0"/>
             <geometry>
-                <box size="1.1 0.1 0.6"/>
+                <box size="0.3 0.3 0.03"/>
+            </geometry>
+        </collision>
+    </link>
+    <joint name="workspace_mount2_joint" type="fixed">
+        <origin xyz="-0.5 0.5 0.85" rpy="0 0 3.14"/>
+        <parent link="$(arg robot_name)_floating_link"/>
+        <child link="workspace_mount2"/>
+    </joint>
+    <joint name="iiwa2_joint" type="fixed">
+        <parent link="workspace_mount2"/>
+        <child link = "iiwa2"/>
+        <origin xyz="0 0 0" rpy="1.57 0 0"/>
+    </joint>
+    <link name="iiwa2">
+        <visual>
+            <origin xyz="0 0 0" rpy="0 0 0"/>
+            <geometry>
+                <mesh filename="package://lbr_description/meshes/envs/visual/iiwa_hande.stl"/>
+            </geometry>
+            <material name="gray">
+                <color rgba="0.7 0.7 0.7 0.2"/>
+            </material>
+        </visual>
+        <collision>
+            <origin xyz="0 0.8 0" rpy="0 0 0"/>
+            <geometry>
+                <box size="0.25 1.5 0.25"/>
             </geometry>
         </collision>
@@ -487,23 +510,23 @@
         </inertial>
     </link>
-    <joint name="frame_joint" type="fixed">
-        <parent link="$(arg robot_name)_floating_link"/>
-        <child link = "frame"/>
-        <origin xyz="-0.2 0.8 0.84" rpy="0 0 0"/>
-    </joint>
-    <link name="frame">
-        <visual>
-            <origin xyz="0 0 0" rpy="0 0 0"/>
-            <geometry>
-                <mesh filename="package://lbr_description/meshes/envs/visual/workspace.stl"/>
-            </geometry>
-            <material name="gray">
-                <color rgba="0.7 0.7 0.7 0.2"/>
-            </material>
-        </visual>
-        <collision>
-            <origin xyz="0 0 -0.4" rpy="0 0 0"/>
-            <geometry>
-                <box size="1.0 1.0 0.7"/>
+    <joint name="softjig_joint" type="fixed">
+        <parent link="frame"/>
+        <child link = "softjig"/>
+        <origin xyz="0.45 0.5 0" rpy="1.57 0 3.14"/>
+    </joint>
+    <link name="softjig">
+        <visual>
+            <origin xyz="0 0 0" rpy="0 0 0"/>
+            <geometry>
+                <mesh filename="package://lbr_description/meshes/envs/visual/softjig.stl"/>
+            </geometry>
+            <material name="dark_gray">
+                <color rgba="0.7 0.7 0.7 1.0"/>
+            </material>
+        </visual>
+        <collision>
+            <origin xyz="0 0 0" rpy="0 0 0"/>
+            <geometry>
+                <mesh filename="package://lbr_description/meshes/envs/collision/softjig.stl"/>
             </geometry>
         </collision>
@@ -517,23 +540,23 @@
         </inertial>
     </link>
-    <joint name="iiwa2_joint" type="fixed">
+    <joint name="round_table_joint" type="fixed">
         <parent link="$(arg robot_name)_floating_link"/>
-        <child link = "iiwa2"/>
-        <origin xyz="-0.005 -0.0045 0.94" rpy="1.57 0 0"/>
-    </joint>
-    <link name="iiwa2">
-        <visual>
-            <origin xyz="0 0 0" rpy="0 0 0"/>
-            <geometry>
-                <mesh filename="package://lbr_description/meshes/envs/visual/iiwa_hande.stl"/>
-            </geometry>
-            <material name="gray">
-                <color rgba="0.7 0.7 0.7 0.2"/>
-            </material>
-        </visual>
-        <collision>
-            <origin xyz="0 0.8 0" rpy="0 0 0"/>
-            <geometry>
-                <box size="0.25 1.5 0.25"/>
+        <child link = "round_table"/>
+        <origin xyz="0 -0.3 0.55" rpy="0 0 0"/>
+    </joint>
+    <link name="round_table">
+        <visual>
+            <origin xyz="0 0 0" rpy="0 0 0"/>
+            <geometry>
+                <cylinder length="0.05" radius="0.43"/>
+            </geometry>
+            <material name="green">
+                <color rgba="0.0 0.8 0.0 0.5"/>
+            </material>
+        </visual>
+        <collision>
+            <origin xyz="0 0 0" rpy="0 0 0"/>
+            <geometry>
+                <cylinder length="0.05" radius="0.43"/>
             </geometry>
         </collision>
@@ -547,23 +570,23 @@
         </inertial>
     </link>
-    <joint name="softjig_joint" type="fixed">
-        <parent link="frame"/>
-        <child link = "softjig"/>
-        <origin xyz="0.45 0 0" rpy="1.57 0 3.14"/>
-    </joint>
-    <link name="softjig">
-        <visual>
-            <origin xyz="0 0 0" rpy="0 0 0"/>
-            <geometry>
-                <mesh filename="package://lbr_description/meshes/envs/visual/softjig.stl"/>
-            </geometry>
-            <material name="dark_gray">
-                <color rgba="0.7 0.7 0.7 1.0"/>
-            </material>
-        </visual>
-        <collision>
-            <origin xyz="0 0 0" rpy="0 0 0"/>
-            <geometry>
-                <mesh filename="package://lbr_description/meshes/envs/collision/softjig.stl"/>
+    <joint name="heater_unit_joint" type="fixed">
+        <parent link="conveyor"/>
+        <child link = "heater_unit"/>
+        <origin xyz="0.242 -1.4 0.8" rpy="0 0 1.57"/>
+    </joint>
+    <link name="heater_unit">
+        <visual>
+            <origin xyz="0 0 0" rpy="0 0 0"/>
+            <geometry>
+                <mesh filename="package://lbr_description/meshes/envs/visual/heater_unit.stl"/>
+            </geometry>
+            <material name="gray">
+                <color rgba="0.7 0.7 0.7 0.2"/>
+            </material>
+        </visual>
+        <collision>
+            <origin xyz="0 0.25 0.32" rpy="0 0 0"/>
+            <geometry>
+                <box size="0.22 0.445 0.4"/>
             </geometry>
         </collision>
@@ -577,64 +600,4 @@
         </inertial>
     </link>
-    <joint name="round_table_joint" type="fixed">
-        <parent link="$(arg robot_name)_floating_link"/>
-        <child link = "round_table"/>
-        <origin xyz="0 -0.7 0.55" rpy="0 0 0"/>
-    </joint>
-    <link name="round_table">
-        <visual>
-            <origin xyz="0 0 0" rpy="0 0 0"/>
-            <geometry>
-                <cylinder length="0.05" radius="0.43"/>
-            </geometry>
-            <material name="green">
-                <color rgba="0.0 0.8 0.0 0.5"/>
-            </material>
-        </visual>
-        <collision>
-            <origin xyz="0 0 0" rpy="0 0 0"/>
-            <geometry>
-                <cylinder length="0.05" radius="0.43"/>
-            </geometry>
-        </collision>
-        <inertial>
-            <origin xyz="0 0 1" rpy="0 0 0"/>
-            <mass value="1"/>
-            <inertia
-                ixx="1.0" ixy="0.0" ixz="0.0"
-                iyy="1.0" iyz="0.0"
-                izz="1.0"/>
-        </inertial>
-    </link>
-    <joint name="heater_unit_joint" type="fixed">
-        <parent link="conveyor"/>
-        <child link = "heater_unit"/>
-        <origin xyz="0.242 -1.4 0.8" rpy="0 0 1.57"/>
-    </joint>
-    <link name="heater_unit">
-        <visual>
-            <origin xyz="0 0 0" rpy="0 0 0"/>
-            <geometry>
-                <mesh filename="package://lbr_description/meshes/envs/visual/heater_unit.stl"/>
-            </geometry>
-            <material name="gray">
-                <color rgba="0.7 0.7 0.7 0.2"/>
-            </material>
-        </visual>
-        <collision>
-            <origin xyz="0 0.25 0.32" rpy="0 0 0"/>
-            <geometry>
-                <box size="0.22 0.445 0.4"/>
-            </geometry>
-        </collision>
-        <inertial>
-            <origin xyz="0 0 1" rpy="0 0 0"/>
-            <mass value="1"/>
-            <inertia
-                ixx="1.0" ixy="0.0" ixz="0.0"
-                iyy="1.0" iyz="0.0"
-                izz="1.0"/>
-        </inertial>
-    </link>
     </xacro:macro>
 </robot>

Commit message: correct environment

File: lbr_description/urdf/iiwa14/iiwa14.xacro (robot description, xacro)
@@ -34,5 +34,5 @@
     </joint>
     <joint name="$(arg robot_name)_joint" type="fixed">
-        <origin xyz="0 0 0.016" rpy="0 0 0.785398"/>
+        <origin xyz="0 0 0.016" rpy="0 0 2.36"/>
         <parent link="workspace_mount1" />
         <child link="$(arg robot_name)_link_0" />

File: lbr_description/urdf/iiwa14/iiwa14_description.xacro (robot description, xacro)
@@ -483,5 +483,5 @@
         <parent link="workspace_mount2"/>
         <child link = "iiwa2"/>
-        <origin xyz="0 0 0" rpy="1.57 0 0"/>
+        <origin xyz="0 0 0" rpy="1.57 0 -2.37"/>
     </joint>
     <link name="iiwa2">
